File: RAK811.sch (KiCad schematic (older format))
At the start: 21 parts, among them P1 CONN_01X02, P2 CONN_01X03, P3 CONN_01X06, P4 CONN_01X14, P5 CONN_01X14, SW1 SW_SPST_Small, U1 RAK811

Commit message: Added IPX + Regulator
Parts:
- removed P4, P5: CONN_01X14, Pin_Headers:Pin_Header_Straight_1x14_Pitch2.54mm, symbol CONN_01X14
- added C6, C7: 22uF, Capacitors_SMD:C_0603, symbol C_Small
- added P4, P5: CONN_01X15, Pin_Headers:Pin_Header_Straight_1x15_Pitch2.54mm, symbol CONN_01X15
- added P6: CONN_01X02, ipx:ipx, symbol CONN_01X02
- added U2: LD1117S12CTR, TO_SOT_Packages_SMD:SOT-223, symbol LD1117S12CTR
- SW1: footprint (none) -> KMR241NG:KMR241NG
Connections:
- net labels added: +5V
- wire segments 108 -> 122
Changed lines of the file:
@@
 LIBS:valves
 LIBS:rak811
-EELAYER 26 0
+LIBS:RAK811-cache
+EELAYER 25 0
 EELAYER END
 $Descr A4 11693 8268
@@
 F 0 "SW1" H 6300 2450 50  0000 L CNN
 F 1 "SW_SPST_Small" H 5900 2550 50  0000 L CNN
-F 2 "" H 6350 2650 50  0001 C CNN
+F 2 "KMR241NG:KMR241NG" H 6350 2650 50  0001 C CNN
 F 3 "" H 6350 2650 50  0000 C CNN
 	1    6350 2650
@@
 Wire Wire Line
 	7600 2100 7200 2100
-$Comp
-L CONN_01X14 P4
-U 1 1 58E85F4E
-P 8600 2650
-F 0 "P4" H 8519 1775 50  0000 C CNN
-F 1 "CONN_01X14" H 8519 1866 50  0000 C CNN
-F 2 "Pin_Headers:Pin_Header_Straight_1x14_Pitch2.54mm" H 8600 2650 50  0001 C CNN
-F 3 "" H 8600 2650 50  0000 C CNN
-	1    8600 2650
-	-1   0    0    1
-$EndComp
 $Comp
 L GND #PWR023
@@
 Text GLabel 8900 3100 2    60   Input ~ 0
 PA15
-$Comp
-L CONN_01X14 P5
-U 1 1 58E86E9C
-P 10350 2650
-F 0 "P5" H 10268 1775 50  0000 C CNN
-F 1 "CONN_01X14" H 10268 1866 50  0000 C CNN
-F 2 "Pin_Headers:Pin_Header_Straight_1x14_Pitch2.54mm" H 10350 2650 50  0001 C CNN
-F 3 "" H 10350 2650 50  0000 C CNN
-	1    10350 2650
-	1    0    0    1
-$EndComp
 $Comp
 L GND #PWR026
@@
 Wire Wire Line
 	6450 1850 6450 1950
+$Comp
+L CONN_01X02 P6
+U 1 1 58ED36C3
+P 1550 1450
+F 0 "P6" H 1469 1175 50  0000 C CNN
+F 1 "CONN_01X02" H 1469 1266 50  0000 C CNN
+F 2 "ipx:ipx" H 1550 1450 50  0001 C CNN
+F 3 "" H 1550 1450 50  0000 C CNN
+	1    1550 1450
+	-1   0    0    1
+$EndComp
+$Comp
+L GND #PWR029
+U 1 1 58ED371F
+P 1850 1400
+F 0 "#PWR029" H 1850 1150 50  0001 C CNN
+F 1 "GND" V 1850 1200 50  0000 C CNN
+F 2 "" H 1850 1400 50  0001 C CNN
+F 3 "" H 1850 1400 50  0001 C CNN
+	1    1850 1400
+	0    -1   -1   0
+$EndComp
+Wire Wire Line
+	1750 1400 1850 1400
+Wire Wire Line
+	2000 1150 2000 1500
+Wire Wire Line
+	2000 1500 1750 1500
+Connection ~ 2000 1150
+$Comp
+L LD1117S12CTR U2
+U 1 1 58ED3B2A
+P 6750 3800
+F 0 "U2" H 6750 4208 50  0000 C CNN
+F 1 "LD1117S12CTR" H 6750 4117 50  0000 C CNN
+F 2 "TO_SOT_Packages_SMD:SOT-223" H 6750 4026 50  0000 C CNN
+F 3 "" H 6750 3800 50  0000 C CNN
+	1    6750 3800
+	1    0    0    -1
+$EndComp
+$Comp
+L C_Small C6
+U 1 1 58ED4012
+P 6300 3900
+F 0 "C6" H 6400 3950 50  0000 L CNN
+F 1 "22uF" H 6400 3850 50  0000 L CNN
+F 2 "Capacitors_SMD:C_0603" H 6300 3900 50  0001 C CNN
+F 3 "" H 6300 3900 50  0001 C CNN
+	1    6300 3900
+	1    0    0    -1
+$EndComp
+$Comp
+L C_Small C7
+U 1 1 58ED4186
+P 7200 3900
+F 0 "C7" H 7300 3950 50  0000 L CNN
+F 1 "22uF" H 7300 3850 50  0000 L CNN
+F 2 "Capacitors_SMD:C_0603" H 7200 3900 50  0001 C CNN
+F 3 "" H 7200 3900 50  0001 C CNN
+	1    7200 3900
+	1    0    0    -1
+$EndComp
+Wire Wire Line
+	7150 3750 7250 3750
+Wire Wire Line
+	7200 3750 7200 3800
+Wire Wire Line
+	6250 3750 6350 3750
+Wire Wire Line
+	6300 3750 6300 3800
+Wire Wire Line
+	6300 4000 6300 4100
+Wire Wire Line
+	6300 4100 7200 4100
+Wire Wire Line
+	7200 4100 7200 4000
+Wire Wire Line
+	6750 4050 6750 4150
+Connection ~ 6750 4100
+$Comp
+L GND #PWR030
+U 1 1 58ED4569
+P 6750 4150
+F 0 "#PWR030" H 6750 3900 50  0001 C CNN
+F 1 "GND" H 6755 3977 50  0000 C CNN
+F 2 "" H 6750 4150 50  0001 C CNN
+F 3 "" H 6750 4150 50  0001 C CNN
+	1    6750 4150
+	1    0    0    -1
+$EndComp
+$Comp
+L +3V3 #PWR031
+U 1 1 58ED47FE
+P 7250 3750
+F 0 "#PWR031" H 7250 3600 50  0001 C CNN
+F 1 "+3V3" V 7250 3900 50  0000 L CNN
+F 2 "" H 7250 3750 50  0000 C CNN
+F 3 "" H 7250 3750 50  0000 C CNN
+	1    7250 3750
+	0    1    1    0
+$EndComp
+$Comp
+L +5V #PWR032
+U 1 1 58ED496B
+P 6250 3750
+F 0 "#PWR032" H 6250 3600 50  0001 C CNN
+F 1 "+5V" V 6265 3878 50  0000 L CNN
+F 2 "" H 6250 3750 50  0000 C CNN
+F 3 "" H 6250 3750 50  0000 C CNN
+	1    6250 3750
+	0    -1   -1   0
+$EndComp
+Connection ~ 6300 3750
+Connection ~ 7200 3750
+$Comp
+L CONN_01X15 P5
+U 1 1 58ED5F7E
+P 10350 2600
+F 0 "P5" H 10428 2641 50  0000 L CNN
+F 1 "CONN_01X15" H 10428 2550 50  0000 L CNN
+F 2 "Pin_Headers:Pin_Header_Straight_1x15_Pitch2.54mm" H 10350 2600 50  0001 C CNN
+F 3 "" H 10350 2600 50  0000 C CNN
+	1    10350 2600
+	1    0    0    -1
+$EndComp
+$Comp
+L CONN_01X15 P4
+U 1 1 58ED60F6
+P 8600 2600
+F 0 "P4" H 8519 1675 50  0000 C CNN
+F 1 "CONN_01X15" H 8519 1766 50  0000 C CNN
+F 2 "Pin_Headers:Pin_Header_Straight_1x15_Pitch2.54mm" H 8600 2600 50  0001 C CNN
+F 3 "" H 8600 2600 50  0000 C CNN
+	1    8600 2600
+	-1   0    0    1
+$EndComp
+Wire Wire Line
+	8800 1900 8850 1900
+Wire Wire Line
+	8850 1900 8850 2000
+Connection ~ 8850 2000
+$Comp
+L +5V #PWR033
+U 1 1 58ED6687
+P 10050 1900
+F 0 "#PWR033" H 10050 1750 50  0001 C CNN
+F 1 "+5V" V 10065 2028 50  0000 L CNN
+F 2 "" H 10050 1900 50  0000 C CNN
+F 3 "" H 10050 1900 50  0000 C CNN
+	1    10050 1900
+	0    -1   -1   0
+$EndComp
+Wire Wire Line
+	10150 1900 10050 1900
 $EndSCHEMATC

Commit message: Added better RF path
Parts:
- removed L1: 10pF C, Capacitors_SMD:C_0603, symbol INDUCTOR_Small
Connections:
- wire segments 122 -> 121
Changed lines of the file:
@@
 L C_Small C3
 U 1 1 58E7D58F
-P 2150 1300
-F 0 "C3" H 1950 1350 50  0000 L CNN
-F 1 "nc" H 1950 1250 50  0000 L CNN
-F 2 "Capacitors_SMD:C_0603" H 2150 1300 50  0001 C CNN
-F 3 "" H 2150 1300 50  0000 C CNN
-	1    2150 1300
-	1    0    0    -1
-$EndComp
-$Comp
-L C_Small C4
-U 1 1 58E7D5CE
-P 2450 1300
-F 0 "C4" H 2350 1250 50  0000 R CNN
-F 1 "nc" H 2358 1345 50  0000 R CNN
-F 2 "Capacitors_SMD:C_0603" H 2450 1300 50  0001 C CNN
-F 3 "" H 2450 1300 50  0000 C CNN
-	1    2450 1300
-	-1   0    0    1
-$EndComp
-$Comp
-L INDUCTOR_Small L1
-U 1 1 58E7D5FC
 P 2300 1150
-F 0 "L1" V 2485 1150 50  0000 C CNN
-F 1 "10pF C" V 2394 1150 50  0000 C CNN
+F 0 "C3" H 2100 1200 50  0000 L CNN
+F 1 "nc" H 2100 1100 50  0000 L CNN
 F 2 "Capacitors_SMD:C_0603" H 2300 1150 50  0001 C CNN
 F 3 "" H 2300 1150 50  0000 C CNN
 	1    2300 1150
-	0    -1   -1   0
-$EndComp
-$Comp
-L GND #PWR013
-U 1 1 58E7DE98
-P 2450 1450
-F 0 "#PWR013" H 2450 1200 50  0001 C CNN
-F 1 "GND" V 2450 1250 50  0000 C CNN
-F 2 "" H 2450 1450 50  0001 C CNN
-F 3 "" H 2450 1450 50  0001 C CNN
-	1    2450 1450
-	1    0    0    -1
-$EndComp
-$Comp
-L GND #PWR014
-U 1 1 58E7DEC6
-P 2150 1450
-F 0 "#PWR014" H 2150 1200 50  0001 C CNN
-F 1 "GND" V 2150 1250 50  0000 C CNN
-F 2 "" H 2150 1450 50  0001 C CNN
-F 3 "" H 2150 1450 50  0001 C CNN
-	1    2150 1450
-	1    0    0    -1
+	0    1    1    0
+$EndComp
+$Comp
+L C_Small C4
+U 1 1 58E7D5CE
+P 2300 1300
+F 0 "C4" H 2200 1250 50  0000 R CNN
+F 1 "nc" H 2208 1345 50  0000 R CNN
+F 2 "Capacitors_SMD:C_0603" H 2300 1300 50  0001 C CNN
+F 3 "" H 2300 1300 50  0000 C CNN
+	1    2300 1300
+	0    -1   -1   0
 $EndComp
 Text GLabel 5150 2600 1    60   Input ~ 0
@@
 Connection ~ 1750 3200
 Wire Wire Line
-	1750 1150 2200 1150
-Wire Wire Line
-	2150 1200 2150 1150
-Connection ~ 2150 1150
-Wire Wire Line
 	2400 1150 2800 1150
 Wire Wire Line
-	2450 1150 2450 1200
+	2450 1150 2450 1300
 Connection ~ 2450 1150
-Wire Wire Line
-	2450 1450 2450 1400
-Wire Wire Line
-	2150 1450 2150 1400
 Wire Wire Line
 	5150 2600 5150 2700
@@
 	1750 1400 1850 1400
 Wire Wire Line
-	2000 1150 2000 1500
-Wire Wire Line
-	2000 1500 1750 1500
-Connection ~ 2000 1150
+	1750 1500 2100 1500
 $Comp
 L LD1117S12CTR U2
@@
 Wire Wire Line
 	10150 1900 10050 1900
+Wire Wire Line
+	1750 1150 2200 1150
+Wire Wire Line
+	2200 1300 2100 1300
+Wire Wire Line
+	2100 1300 2100 1500
+Wire Wire Line
+	2450 1300 2400 1300
 $EndSCHEMATC
