File: RAK811.sch (KiCad schematic (older format))
At the start: 24 parts, among them P1 CONN_01X02, P2 CONN_01X03, P3 CONN_01X06, P4 CONN_01X15, P5 CONN_01X15, P6 CONN_01X02, SW1 SW_SPST_Small, U1 RAK811, U2 LD1117S12CTR

Commit message: rak811_breakout: Update to V2.1
Parts:
- C1, C2, C3, C4, C5, C6, C7: symbol C_Small -> device:C_Small
- D1, D2: symbol LED -> device:LED
- P1, P6: symbol CONN_01X02 -> Connector:Conn_01x02
- P2: symbol CONN_01X03 -> Connector:Conn_01x03
- P3: symbol CONN_01X06 -> Connector:Conn_01x06
- P4, P5: symbol CONN_01X15 -> Connector:Conn_01x15
- R1, R2, R3, R4, R5, R6: symbol R_Small -> device:R_Small
- SW1: symbol SW_SPST_Small -> Switch:SW_SPST
- U1: symbol RAK811 -> rak811:RAK811
- U2: symbol LD1117S12CTR -> regul:AP1117-15
Connections:
- wire segments 121 -> 135
